File: pcb/CarDisplay/CarDisplay.kicad_sch (KiCad schematic)
At the start: 11 parts, among them J1 Switch, J2 Display1, J3 Display2, J4 ECU_RS232, J5 SpeedSensor, U1 MAX3232

Commit message: pcb dev
Parts:
- added R1, R2: 22R, Resistor_SMD:R_0805_2012Metric_Pad1.20x1.40mm_HandSolder, symbol Device:R_Small
Connections:
- net at XA1.D11 (D11_MOSI): now also R1.1
- net at XA1.D13 (D13_SCK): now also R2.1
Changed lines of the file:
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@@
 (kicad_sch (version 20230121) (generator eeschema)
   (paper "A4")
+  (wire (pts (xy 104.14 82.55) (xy 113.03 82.55))
+    (stroke (width 0) (type default))
+  )
+  (wire (pts (xy 104.14 87.63) (xy 110.49 87.63))
+    (stroke (width 0) (type default))
+  )
+  (wire (pts (xy 110.49 90.17) (xy 113.03 90.17))
+    (stroke (width 0) (type default))
+  )
+  (wire (pts (xy 110.49 87.63) (xy 110.49 90.17))
+    (stroke (width 0) (type default))
+  )
   (symbol (lib_id "Interface_UART:MAX3232") (at 160.02 82.55 0) (unit 1)
     (in_bom yes) (on_board yes) (dnp no) (fields_autoplaced)
@@
     )
   )
+  (symbol (lib_id "Device:R_Small") (at 115.57 82.55 90) (unit 1)
+    (in_bom yes) (on_board yes) (dnp no) (fields_autoplaced)
+    (property "Reference" "R1" (at 115.57 77.6691 90)
+      (effects (font (size 1.27 1.27)))
+    )
+    (property "Value" "22R" (at 115.57 80.0933 90)
+      (effects (font (size 1.27 1.27)))
+    )
+    (property "Footprint" "Resistor_SMD:R_0805_2012Metric_Pad1.20x1.40mm_HandSolder" (at 115.57 82.55 0)
+      (effects (font (size 1.27 1.27)) hide)
+    )
+    (property "Datasheet" "~" (at 115.57 82.55 0)
+      (effects (font (size 1.27 1.27)) hide)
+    )
+    (pin "1")
+    (pin "2")
+    (instances
+      (project "CarDisplay"
+        (path "/6780f1c0-9a73-40a2-8ba0-13c7b9c3b1ed"
+          (reference "R1") (unit 1)
+        )
+      )
+    )
+  )
   (symbol (lib_id "Connector:DE9_Receptacle") (at 226.06 76.2 0) (unit 1)
     (in_bom yes) (on_board yes) (dnp no) (fields_autoplaced)
@@
         )
       )
+    )
+  )
+  (symbol (lib_id "Device:R_Small") (at 115.57 90.17 90) (unit 1)
+    (in_bom yes) (on_board yes) (dnp no) (fields_autoplaced)
+    (property "Reference" "R2" (at 115.57 85.2891 90)
+      (effects (font (size 1.27 1.27)))
+    )
+    (property "Value" "22R" (at 115.57 87.7133 90)
+      (effects (font (size 1.27 1.27)))
+    )
+    (property "Footprint" "Resistor_SMD:R_0805_2012Metric_Pad1.20x1.40mm_HandSolder" (at 115.57 90.17 0)
+      (effects (font (size 1.27 1.27)) hide)
+    )
+    (property "Datasheet" "~" (at 115.57 90.17 0)
+      (effects (font (size 1.27 1.27)) hide)
+    )
+    (pin "1")
+    (pin "2")
+    (instances
+      (project "CarDisplay"
+        (path "/6780f1c0-9a73-40a2-8ba0-13c7b9c3b1ed"
+          (reference "R2") (unit 1)
+        )
+      )

Commit message: pcb dev
Parts:
- added C1, C2: 100nF, Capacitor_SMD:C_1206_3216Metric_Pad1.33x1.80mm_HandSolder, symbol Device:C_Small
- added C3: C_Polarized, symbol Device:C_Polarized
- added D1: BZT52Bxx, Diode_SMD:D_SOD-123F, symbol Diode:BZT52Bxx
- added R10, R9: 4k7, Resistor_SMD:R_0805_2012Metric_Pad1.20x1.40mm_HandSolder, symbol Device:R_Small
- added R11, R3, R4, R5, R6: 22R, Resistor_SMD:R_0805_2012Metric_Pad1.20x1.40mm_HandSolder, symbol Device:R_Small
- added R12, R13: 0R, Resistor_SMD:R_0805_2012Metric_Pad1.20x1.40mm_HandSolder, symbol Device:R_Small
- added R7, R8: 0R / NC, Resistor_SMD:R_0805_2012Metric_Pad1.20x1.40mm_HandSolder, symbol Device:R_Small
Connections:
- net at U1.11 (T1IN): now also R12.2
- net at U1.12 (R1OUT): now also R13.2
- net ECU_TX: now reaches U1.13 (R1IN)
- net ECU_TX: now also J4.3
- net ECU_RX: now reaches U1.14 (T1OUT)
- net ECU_RX: now also J4.2
- net GND: now reaches U1.15 (GND)
- net GND: now also J1.2 (Pin_2), J3.5 (Pin_5), J4.5, J5.3 (Pin_3), XA1.GND1 (GND), XA1.GND2 (GND), C1.2, C2.2, C3.2, D1.2 (A)
- net +5V: now reaches U1.16 (VCC)
- net +5V: now also J4.1, J5.1 (Pin_1), XA1.5V, C2.1, C3.1, R7.1
- net DISP_CLK: now reaches J2.1 (Pin_1)
- net DISP_CLK: now also R2.2
- net DISP_DIN: now reaches J2.2 (Pin_2)
- net DISP_DIN: now also R1.2
- net DISP_CS: now reaches J2.3 (Pin_3)
- net DISP_CS: now also R3.1
- net at J1.1 (Pin_1): now also D1.1 (K), R10.2, R9.2
- net at J5.2 (Pin_2): now also R11.2
- net DISP_RST: now reaches J3.1 (Pin_1)
- net DISP_RST: now also R6.2
- net DISP_DC: now reaches J3.2 (Pin_2)
- net DISP_DC: now also R4.2
- net at J3.3 (Pin_3): now also R7.2, R8.2
- net DISP_BL: now reaches J3.4 (Pin_4)
- net DISP_BL: now also R5.2
- net +3.3V: now reaches XA1.3V3 (3.3V)
- net +3.3V: now also R10.1, R8.1
- net UART_PC_RX: now reaches XA1.A2
- net at XA1.A3: now also R3.2
- net UART_PC_TX: now reaches XA1.A7
- net UART_ECU_RX: now reaches XA1.D0 (D0_RX0)
- net UART_ECU_RX: now also R13.1
- net UART_ECU_TX: now reaches XA1.D1 (D1_TX0)
- net UART_ECU_TX: now also R12.1
- net at XA1.D2: now also R5.1
- net at XA1.D3: now also R6.1
- net at XA1.D4: now also R4.1
- net SPEED_SENS: now reaches XA1.D9
- net SPEED_SENS: now also R11.1
- new net SWITCH: C1.1, R9.1
- no-connect marks 0 -> 19
Other:
- note added: "Choose 5V or 3.3V"
- moved on the sheet: J1, J2, J3, J4, J5, R1, R2, U1, XA1

Commit message: pcb dev
Parts:
- removed J4: ECU_RS232, Connector_Dsub:DSUB-9_Female_Horizontal_P2.77x2.84mm_EdgePinOffset4.94mm_Housed_MountingHolesOffset7.48mm, symbol Connector:DE9_Receptacle
- added C10, C11, C12, C4, C5, C6, C7, C8, C9: 100nF, Capacitor_SMD:C_1206_3216Metric_Pad1.33x1.80mm_HandSolder, symbol Device:C_Small
- added J6: ECU, _MyFootprints:15EDGVC-3.5-05P, symbol Connector_Generic:Conn_01x05
- added R14, R15, R16, R17: 0R / NC, Resistor_SMD:R_0805_2012Metric_Pad1.20x1.40mm_HandSolder, symbol Device:R_Small
- C3: value C_Polarized -> 100u; footprint (none) -> _MyFootprints:CP_LYING_11x6_2,5mm
Connections:
- net +3.3V: now also C10.1, R15.1, R17.1
- net +5V: now also C11.1, J6.2 (Pin_2), R14.1, R16.1; no longer J5.1 (Pin_1), U1.16 (VCC)
- net DISP_BL: now also J3.5 (Pin_5); no longer J3.4 (Pin_4)
- net ECU_RX: now also J6.5 (Pin_5)
- net ECU_TX: now also J6.4 (Pin_4)
- net GND: now also J3.4 (Pin_4), J5.2 (Pin_2), U1.10 (T2IN), U1.8 (R2IN), C10.2, C11.2, C12.2, C4.2, C7.2, C8.2, C9.2, J6.1 (Pin_1); no longer J3.5 (Pin_5), J5.3 (Pin_3)
- net SPEED_SENS: now also R11.2; no longer R11.1
- net SWITCH: now also XA1.D6
- net at U1.1 (C1+): now also C5.1
- net at U1.2 (VS+): now also C7.1
- net at U1.3 (C1-): now also C5.2
- net at U1.4 (C2+): now also C6.1
- net at U1.5 (C2-): now also C6.2
- net at U1.6 (VS-): now also C8.1
- net at J3.3 (Pin_3), R7.2, R8.2: now also C12.1
- new net: C4.1, R14.2, R15.2, U1.16 (VCC)
- new net: C9.1, J5.1 (Pin_1), R16.2, R17.2
- new net: J5.3 (Pin_3), R11.1
- no-connect marks 19 -> 17
Other:
- company: (none) -> GruzaiGarage
- title: (none) -> CarDisplay
- moved on the sheet: J2, J3, R11, R12, R13, R7, R8, U1

Commit message: pcb dev, looking for better connectors
Parts:
- removed J6: ECU, _MyFootprints:15EDGVC-3.5-05P, symbol Connector_Generic:Conn_01x05
- added J4: ECU, Connector_Dsub:DSUB-9_Female_Horizontal_P2.77x2.84mm_EdgePinOffset4.94mm_Housed_MountingHolesOffset7.48mm, symbol Connector:DE9_Plug_MountingHoles
- added R18, R19: 22R, Resistor_SMD:R_0805_2012Metric_Pad1.20x1.40mm_HandSolder, symbol Device:R_Small
Connections:
- net +5V: now also J4.1
- net ECU_RX: now also R18.1
- net ECU_TX: now also R19.1
- net GND: now also J4.5
- new net: J4.3, R19.2
- new net: J4.2, R18.2
- no-connect marks 17 -> 22
Other:
- moved on the sheet: C2, C3

Commit message: readme
Parts:
- removed J1: Switch, _MyFootprints:15EDGVC-3.5-02P, symbol Connector_Generic:Conn_01x02
- removed J2: Display1, _MyFootprints:15EDGVC-3.5-03P, symbol Connector_Generic:Conn_01x03
- removed J3: Display2, _MyFootprints:15EDGVC-3.5-05P, symbol Connector_Generic:Conn_01x05
- removed J5: SpeedSensor, _MyFootprints:15EDGVC-3.5-03P, symbol Connector_Generic:Conn_01x03
- added J2: DISPLAY, Connector_Molex:Molex_Mini-Fit_Jr_5569-08A2_2x04_P4.20mm_Horizontal, symbol Connector_Generic:Conn_01x08
- added J3: SWITCH&SPEEDSENS, Connector_Molex:Molex_Mini-Fit_Jr_5569-06A2_2x03_P4.20mm_Horizontal, symbol Connector_Generic:Conn_01x06
- C3: footprint _MyFootprints:CP_LYING_11x6_2,5mm -> _MyFootprints:CP_LYING_16x10_5,0mm
- renumbered J4 to J1
Connections:
- net DISP_BL: now also J2.8 (Pin_8)
- net DISP_CLK: now also J2.1 (Pin_1)
- net DISP_CS: now also J2.3 (Pin_3)
- net DISP_DC: now also J2.5 (Pin_5)
- net DISP_DIN: now also J2.2 (Pin_2)
- net DISP_RST: now also J2.4 (Pin_4)
- net GND: now also J2.7 (Pin_7), J3.2 (Pin_2), J3.6 (Pin_6)
- net at D1.1 (K), R10.2, R9.2: now also J3.5 (Pin_5)
- net at C9.1, R16.2, R17.2: now also J3.1 (Pin_1)
- net at C12.1, R7.2, R8.2: now also J2.6 (Pin_6)
- net at R11.1: now also J3.3 (Pin_3)
- no-connect marks 22 -> 23
Other:
- moved on the sheet: C1, D1, R10, R9

Commit message: pcb finished
Parts:
- added J4, J6: RX, _MyFootprints:MeasuringPin, symbol Connector_Generic:Conn_01x01
- added J5, J7: TX, _MyFootprints:MeasuringPin, symbol Connector_Generic:Conn_01x01
- added J8: GND, _MyFootprints:MeasuringPin, symbol Connector_Generic:Conn_01x01
Connections:
- net DISP_BL: now also J2.7 (Pin_7); no longer J2.8 (Pin_8)
- net DISP_CLK: now also J2.8 (Pin_8); no longer J2.1 (Pin_1)
- net DISP_CS: now also J2.4 (Pin_4); no longer J2.3 (Pin_3)
- net DISP_DC: now also J2.6 (Pin_6); no longer J2.5 (Pin_5)
- net DISP_RST: now also J2.3 (Pin_3); no longer J2.4 (Pin_4)
- net ECU_RX: now also J4.1 (Pin_1)
- net ECU_TX: now also J5.1 (Pin_1)
- net GND: now also J2.1 (Pin_1), J3.5 (Pin_5), J8.1 (Pin_1); no longer J2.7 (Pin_7), J3.6 (Pin_6), XA1.GND1 (GND)
- net UART_ECU_RX: now also J6.1 (Pin_1)
- net UART_ECU_TX: now also J7.1 (Pin_1)
- net at D1.1 (K), R10.2, R9.2: now also J3.6 (Pin_6); no longer J3.5 (Pin_5)
- net at C12.1, R7.2, R8.2: now also J2.5 (Pin_5); no longer J2.6 (Pin_6)
- no-connect marks 23 -> 24
Other:
- moved on the sheet: C12, R7, R8
