File: pcb/CarDisplay/CarDisplay.kicad_pcb (KiCad board)
At the start: 2 copper layers, 52.5 x 55 mm, 11 parts, among them J1 Switch, J2 Display1, J3 Display2, J4 ECU_RS232, J5 SpeedSensor, U1 MAX3232

Commit message: pcb dev
Parts:
- moved H2 65.6 mm to (92.0, 19.5)
- moved H4 62.0 mm to (92.0, 81.5)
- moved H3 29.9 mm to (47.5, 81.5)
- moved H1 24.2 mm to (47.5, 19.5)
Other:
- board size 52.5 x 55 mm -> 52.5 x 70 mm
Changed lines of the file:
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@@
   (net 68 "unconnected-(J5-Pin_3-Pad3)")
   (footprint "MountingHole:MountingHole_3.5mm" (layer "F.Cu")
-    (at 32.5 55.6)
+    (at 47.5 81.5)
     (descr "Mounting Hole 3.5mm, no annular")
     (tags "mounting hole 3.5mm no annular")
@@
     (property "ki_keywords" "mounting hole")
     (attr exclude_from_pos_files)
-    (fp_text reference "H3" (at 0 -4.5) (layer "F.SilkS")
-        (effects (font (size 1 1) (thickness 0.15)))
-    )
-    (fp_text value "MountingHole" (at 0 4.5) (layer "F.Fab")
+    (fp_text reference "H3" (at 0 -4.5) (layer "F.SilkS") hide
+        (effects (font (size 1 1) (thickness 0.15)))
+    )
+    (fp_text value "MountingHole" (at 0 4.5) (layer "F.Fab") hide
         (effects (font (size 1 1) (thickness 0.15)))
     )
@@
   )
   (footprint "MountingHole:MountingHole_3.5mm" (layer "F.Cu")
-    (at 32.5 47.05)
+    (at 92 19.5)
     (descr "Mounting Hole 3.5mm, no annular")
     (tags "mounting hole 3.5mm no annular")
@@
     (property "ki_keywords" "mounting hole")
     (attr exclude_from_pos_files)
-    (fp_text reference "H2" (at 0 -4.5) (layer "F.SilkS")
-        (effects (font (size 1 1) (thickness 0.15)))
-    )
-    (fp_text value "MountingHole" (at 0 4.5) (layer "F.Fab")
+    (fp_text reference "H2" (at 0 -4.5) (layer "F.SilkS") hide
+        (effects (font (size 1 1) (thickness 0.15)))
+    )
+    (fp_text value "MountingHole" (at 0 4.5) (layer "F.Fab") hide
         (effects (font (size 1 1) (thickness 0.15)))
     )
@@
   )
   (footprint "MountingHole:MountingHole_3.5mm" (layer "F.Cu")
-    (at 32.5 64.15)
+    (at 92 81.5)
     (descr "Mounting Hole 3.5mm, no annular")
     (tags "mounting hole 3.5mm no annular")
@@
     (property "ki_keywords" "mounting hole")
     (attr exclude_from_pos_files)
-    (fp_text reference "H4" (at 0 -4.5) (layer "F.SilkS")
-        (effects (font (size 1 1) (thickness 0.15)))
-    )
-    (fp_text value "MountingHole" (at 0 4.5) (layer "F.Fab")
+    (fp_text reference "H4" (at 0 -4.5) (layer "F.SilkS") hide
+        (effects (font (size 1 1) (thickness 0.15)))
+    )
+    (fp_text value "MountingHole" (at 0 4.5) (layer "F.Fab") hide
         (effects (font (size 1 1) (thickness 0.15)))
     )
@@
   )
   (footprint "MountingHole:MountingHole_3.5mm" (layer "F.Cu")
-    (at 32.5 38.5)
+    (at 47.5 19.5)
     (descr "Mounting Hole 3.5mm, no annular")
     (tags "mounting hole 3.5mm no annular")
@@
     (property "ki_keywords" "mounting hole")
     (attr exclude_from_pos_files)
-    (fp_text reference "H1" (at 0 -4.5) (layer "F.SilkS")
-        (effects (font (size 1 1) (thickness 0.15)))
-    )
-    (fp_text value "MountingHole" (at 0 4.5) (layer "F.Fab")
+    (fp_text reference "H1" (at 0 -4.5) (layer "F.SilkS") hide
+        (effects (font (size 1 1) (thickness 0.15)))
+    )
+    (fp_text value "MountingHole" (at 0 4.5) (layer "F.Fab") hide
         (effects (font (size 1 1) (thickness 0.15)))
     )
@@
     (property "ki_keywords" "connector")
     (attr smd)
-    (fp_text reference "J1" (at -3 2 180 unlocked) (layer "B.SilkS")
+    (fp_text reference "J1" (at -3 2 180 unlocked) (layer "B.SilkS") hide
         (effects (font (size 0.5 0.5) (thickness 0.125)) (justify mirror))
     )
-    (fp_text value "Switch" (at 0 -6.5 180 unlocked) (layer "B.Fab")
-        (effects (font (size 0.5 0.5) (thickness 0.125)) (justify mirror))
+    (fp_text value "Switch" (at 0 -1.75 270 unlocked) (layer "F.SilkS")
+        (effects (font (size 1 1) (thickness 0.2) bold))
     )
     (fp_line (start -3 1) (end -3 -4.5)
@@
     (property "ki_keywords" "connector")
     (attr smd)
-    (fp_text reference "J3" (at 0 2 180 unlocked) (layer "B.SilkS")
+    (fp_text reference "J3" (at 0 2 180 unlocked) (layer "B.SilkS") hide
         (effects (font (size 0.5 0.5) (thickness 0.125)) (justify mirror))
     )
-    (fp_text value "Display2" (at 0 -16.5 180 unlocked) (layer "B.Fab")
-        (effects (font (size 0.5 0.5) (thickness 0.125)) (justify mirror))
+    (fp_text value "Display2" (at 0 -7 270 unlocked) (layer "F.SilkS")
+        (effects (font (size 1 1) (thickness 0.2) bold))
     )
     (fp_line (start -3 1) (end -3 -15)
@@
     (property "ki_keywords" "connector")
     (attr smd)
-    (fp_text reference "J2" (at 0 2.5 180 unlocked) (layer "B.SilkS")
+    (fp_text reference "J2" (at 0 2.5 180 unlocked) (layer "B.SilkS") hide
         (effects (font (size 0.5 0.5) (thickness 0.125)) (justify mirror))
     )
-    (fp_text value "Display1" (at 0 -9 180 unlocked) (layer "B.Fab")
-        (effects (font (size 0.5 0.5) (thickness 0.125)) (justify mirror))
+    (fp_text value "Display1" (at 0 -3.5 270 unlocked) (layer "F.SilkS")
+        (effects (font (size 1 1) (thickness 0.2) bold))
     )
     (fp_line (start -3 1) (end -3 -8)
@@
     (property "ki_keywords" "connector")
     (attr smd)
-    (fp_text reference "J5" (at 0 2.5 180 unlocked) (layer "B.SilkS")
+    (fp_text reference "J5" (at 0 2.5 180 unlocked) (layer "B.SilkS") hide
         (effects (font (size 0.5 0.5) (thickness 0.125)) (justify mirror))
     )
-    (fp_text value "SpeedSensor" (at 0 -9 180 unlocked) (layer "B.Fab")
-        (effects (font (size 0.5 0.5) (thickness 0.125)) (justify mirror))
+    (fp_text value "SpeedSensor" (at 0 -3.5 270 unlocked) (layer "F.SilkS")
+        (effects (font (size 1 1) (thickness 0.2) bold))
     )
     (fp_line (start -3 1) (end -3 -8)
@@
     )
   )
-  (gr_line (start 96 23) (end 43.5 23)
-    (stroke (width 0.1) (type default)) (layer "Edge.Cuts"))
-  (gr_line (start 43.5 23) (end 43.5 78)
-    (stroke (width 0.1) (type default)) (layer "Edge.Cuts"))
-  (gr_line (start 96 78) (end 96 23)
-    (stroke (width 0.1) (type default)) (layer "Edge.Cuts"))
-  (gr_line (start 43.5 78) (end 96 78)
+  (gr_line (start 94.5 15.5) (end 45 15.5)
+    (stroke (width 0.1) (type default)) (layer "Edge.Cuts"))
+  (gr_arc (start 43.5 17) (mid 43.93934 15.93934) (end 45 15.5)
+    (stroke (width 0.1) (type default)) (layer "Edge.Cuts"))
+  (gr_arc (start 94.5 15.5) (mid 95.56066 15.93934) (end 96 17)
+    (stroke (width 0.1) (type default)) (layer "Edge.Cuts"))
+  (gr_line (start 43.5 17) (end 43.5 84)
+    (stroke (width 0.1) (type default)) (layer "Edge.Cuts"))
+  (gr_arc (start 96 84) (mid 95.56066 85.06066) (end 94.5 85.5)
+    (stroke (width 0.1) (type default)) (layer "Edge.Cuts"))
+  (gr_line (start 96 84) (end 96 17)
+    (stroke (width 0.1) (type default)) (layer "Edge.Cuts"))
+  (gr_arc (start 45 85.5) (mid 43.93934 85.06066) (end 43.5 84)
+    (stroke (width 0.1) (type default)) (layer "Edge.Cuts"))
+  (gr_line (start 45 85.5) (end 94.5 85.5)
     (stroke (width 0.1) (type default)) (layer "Edge.Cuts"))
 )

Commit message: pcb dev
Parts:
- added R1: 22R, Resistor_SMD:R_0805_2012Metric_Pad1.20x1.40mm_HandSolder, B.Cu at (73.5, 64.5)
- added R2: 22R, Resistor_SMD:R_0805_2012Metric_Pad1.20x1.40mm_HandSolder, B.Cu at (81.0, 67.5)
Connections:
- XA1 pad D11: unconnected-(XA1-D11_MOSI-PadD11) -> Net-(XA1-D11_MOSI)
- XA1 pad D13: unconnected-(XA1-D13_SCK-PadD13) -> Net-(XA1-D13_SCK)
Changed lines of the file:
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@@
   (net 56 "unconnected-(XA1-PadD9)")
   (net 57 "unconnected-(XA1-PadD10)")
-  (net 58 "unconnected-(XA1-D11_MOSI-PadD11)")
+  (net 58 "Net-(XA1-D11_MOSI)")
   (net 59 "unconnected-(XA1-D12_MISO-PadD12)")
-  (net 60 "unconnected-(XA1-D13_SCK-PadD13)")
+  (net 60 "unconnected-(R1-Pad2)")
   (net 61 "unconnected-(XA1-GND-PadGND1)")
   (net 62 "unconnected-(XA1-GND-PadGND2)")
@@
   (net 67 "unconnected-(J5-Pin_2-Pad2)")
   (net 68 "unconnected-(J5-Pin_3-Pad3)")
+  (net 69 "Net-(XA1-D13_SCK)")
+  (net 70 "unconnected-(R2-Pad2)")
   (footprint "MountingHole:MountingHole_3.5mm" (layer "F.Cu")
     (at 47.5 81.5)
@@
       (net 57 "unconnected-(XA1-PadD10)") (pinfunction "D10") (pintype "bidirectional"))
     (pad "D11" thru_hole circle (at -7.62 -6.35) (size 1.7272 1.7272) (drill 1.016) (layers "*.Cu" "*.Mask")
-      (net 58 "unconnected-(XA1-D11_MOSI-PadD11)") (pinfunction "D11_MOSI") (pintype "bidirectional"))
+      (net 58 "Net-(XA1-D11_MOSI)") (pinfunction "D11_MOSI") (pintype "bidirectional"))
     (pad "D12" thru_hole circle (at -7.62 -3.81) (size 1.7272 1.7272) (drill 1.016) (layers "*.Cu" "*.Mask")
       (net 59 "unconnected-(XA1-D12_MISO-PadD12)") (pinfunction "D12_MISO") (pintype "bidirectional"))
     (pad "D13" thru_hole circle (at 7.62 -3.81) (size 1.7272 1.7272) (drill 1.016) (layers "*.Cu" "*.Mask")
-      (net 60 "unconnected-(XA1-D13_SCK-PadD13)") (pinfunction "D13_SCK") (pintype "bidirectional"))
+      (net 69 "Net-(XA1-D13_SCK)") (pinfunction "D13_SCK") (pintype "bidirectional"))
     (pad "GND1" thru_hole rect (at -7.62 -31.75) (size 1.7272 1.7272) (drill 1.016) (layers "*.Cu" "*.Mask")
       (net 61 "unconnected-(XA1-GND-PadGND1)") (pinfunction "GND") (pintype "power_in"))
@@
       (scale (xyz 1 1 1))
       (rotate (xyz 90 180 -90))
+    )
+  )
+  (footprint "Resistor_SMD:R_0805_2012Metric_Pad1.20x1.40mm_HandSolder" (layer "B.Cu")
+    (at 81 67.5 180)
+    (descr "Resistor SMD 0805 (2012 Metric), square (rectangular) end terminal, IPC_7351 nominal with elongated pad for handsoldering. (Body size source: IPC-SM-782 page 72, https://www.pcb-3d.com/wordpress/wp-content/uploads/ipc-sm-782a_amendment_1_and_2.pdf), generated with kicad-footprint-generator")
+    (tags "resistor handsolder")
+    (property "Sheetfile" "CarDisplay.kicad_sch")
+    (property "Sheetname" "")
+    (property "ki_description" "Resistor, small symbol")
+    (property "ki_keywords" "R resistor")
+    (attr smd)
+    (fp_text reference "R2" (at 0 1.65) (layer "B.SilkS")
+        (effects (font (size 1 1) (thickness 0.15)) (justify mirror))
+    )
+    (fp_text value "22R" (at 0 -1.65) (layer "B.Fab")
+        (effects (font (size 1 1) (thickness 0.15)) (justify mirror))
+    )
+    (fp_text user "${REFERENCE}" (at 0 0) (layer "B.Fab")
+        (effects (font (size 0.5 0.5) (thickness 0.08)) (justify mirror))
+    )
+    (fp_line (start -0.227064 -0.735) (end 0.227064 -0.735)
+      (stroke (width 0.12) (type solid)) (layer "B.SilkS"))
+    (fp_line (start -0.227064 0.735) (end 0.227064 0.735)
+      (stroke (width 0.12) (type solid)) (layer "B.SilkS"))
+    (fp_line (start -1.85 -0.95) (end -1.85 0.95)
+      (stroke (width 0.05) (type solid)) (layer "B.CrtYd"))
+    (fp_line (start -1.85 0.95) (end 1.85 0.95)
+      (stroke (width 0.05) (type solid)) (layer "B.CrtYd"))
+    (fp_line (start 1.85 -0.95) (end -1.85 -0.95)
+      (stroke (width 0.05) (type solid)) (layer "B.CrtYd"))
+    (fp_line (start 1.85 0.95) (end 1.85 -0.95)
+      (stroke (width 0.05) (type solid)) (layer "B.CrtYd"))
+    (fp_line (start -1 -0.625) (end -1 0.625)
+      (stroke (width 0.1) (type solid)) (layer "B.Fab"))
+    (fp_line (start -1 0.625) (end 1 0.625)
+      (stroke (width 0.1) (type solid)) (layer "B.Fab"))
+    (fp_line (start 1 -0.625) (end -1 -0.625)
+      (stroke (width 0.1) (type solid)) (layer "B.Fab"))
+    (fp_line (start 1 0.625) (end 1 -0.625)
+      (stroke (width 0.1) (type solid)) (layer "B.Fab"))
+    (pad "1" smd roundrect (at -1 0 180) (size 1.2 1.4) (layers "B.Cu" "B.Paste" "B.Mask") (roundrect_rratio 0.208333)
+      (net 69 "Net-(XA1-D13_SCK)") (pintype "passive"))
+    (pad "2" smd roundrect (at 1 0 180) (size 1.2 1.4) (layers "B.Cu" "B.Paste" "B.Mask") (roundrect_rratio 0.208333)
+      (net 70 "unconnected-(R2-Pad2)") (pintype "passive"))
+    (model "${KICAD6_3DMODEL_DIR}/Resistor_SMD.3dshapes/R_0805_2012Metric.wrl"
+      (offset (xyz 0 0 0))
+      (scale (xyz 1 1 1))
+      (rotate (xyz 0 0 0))
     )
   )
@@
       (offset (xyz 0 0 0))
       (scale (xyz 1 1 1))
+      (rotate (xyz 0 0 0))
+    )
+  )
+  (footprint "Resistor_SMD:R_0805_2012Metric_Pad1.20x1.40mm_HandSolder" (layer "B.Cu")
+    (at 73.5 64.5)
+    (descr "Resistor SMD 0805 (2012 Metric), square (rectangular) end terminal, IPC_7351 nominal with elongated pad for handsoldering. (Body size source: IPC-SM-782 page 72, https://www.pcb-3d.com/wordpress/wp-content/uploads/ipc-sm-782a_amendment_1_and_2.pdf), generated with kicad-footprint-generator")
+    (tags "resistor handsolder")
+    (property "Sheetfile" "CarDisplay.kicad_sch")
+    (property "Sheetname" "")
+    (property "ki_description" "Resistor, small symbol")
+    (property "ki_keywords" "R resistor")
+    (attr smd)
+    (fp_text reference "R1" (at 0 1.65) (layer "B.SilkS")
+        (effects (font (size 1 1) (thickness 0.15)) (justify mirror))
+    )
+    (fp_text value "22R" (at 0 -1.65) (layer "B.Fab")
+        (effects (font (size 1 1) (thickness 0.15)) (justify mirror))
+    )
+    (fp_text user "${REFERENCE}" (at 0 0) (layer "B.Fab")
+        (effects (font (size 0.5 0.5) (thickness 0.08)) (justify mirror))
+    )
+    (fp_line (start -0.227064 -0.735) (end 0.227064 -0.735)
+      (stroke (width 0.12) (type solid)) (layer "B.SilkS"))
+    (fp_line (start -0.227064 0.735) (end 0.227064 0.735)
+      (stroke (width 0.12) (type solid)) (layer "B.SilkS"))
+    (fp_line (start -1.85 -0.95) (end -1.85 0.95)
+      (stroke (width 0.05) (type solid)) (layer "B.CrtYd"))
+    (fp_line (start -1.85 0.95) (end 1.85 0.95)
+      (stroke (width 0.05) (type solid)) (layer "B.CrtYd"))
+    (fp_line (start 1.85 -0.95) (end -1.85 -0.95)
+      (stroke (width 0.05) (type solid)) (layer "B.CrtYd"))
+    (fp_line (start 1.85 0.95) (end 1.85 -0.95)
+      (stroke (width 0.05) (type solid)) (layer "B.CrtYd"))
+    (fp_line (start -1 -0.625) (end -1 0.625)
+      (stroke (width 0.1) (type solid)) (layer "B.Fab"))
+    (fp_line (start -1 0.625) (end 1 0.625)
+      (stroke (width 0.1) (type solid)) (layer "B.Fab"))
+    (fp_line (start 1 -0.625) (end -1 -0.625)
+      (stroke (width 0.1) (type solid)) (layer "B.Fab"))
+    (fp_line (start 1 0.625) (end 1 -0.625)
+      (stroke (width 0.1) (type solid)) (layer "B.Fab"))
+    (pad "1" smd roundrect (at -1 0) (size 1.2 1.4) (layers "B.Cu" "B.Paste" "B.Mask") (roundrect_rratio 0.208333)
+      (net 58 "Net-(XA1-D11_MOSI)") (pintype "passive"))
+    (pad "2" smd roundrect (at 1 0) (size 1.2 1.4) (layers "B.Cu" "B.Paste" "B.Mask") (roundrect_rratio 0.208333)
+      (net 60 "unconnected-(R1-Pad2)") (pintype "passive"))
+    (model "${KICAD6_3DMODEL_DIR}/Resistor_SMD.3dshapes/R_0805_2012Metric.wrl"
+      (offset (xyz 0 0 0))
+      (scale (xyz 1 1 1))

Commit message: pcb dev
Parts:
- removed J4: ECU_RS232, Connector_Dsub:DSUB-9_Female_Horizontal_P2.77x2.84mm_EdgePinOffset4.94mm_Housed_MountingHolesOffset7.48mm
- added C1: 100nF, Capacitor_SMD:C_1206_3216Metric_Pad1.33x1.80mm_HandSolder, B.Cu at (72.5, 49.0)
- added C10: 100nF, Capacitor_SMD:C_1206_3216Metric_Pad1.33x1.80mm_HandSolder, B.Cu at (79.0, 64.0)
- added C11: 100nF, Capacitor_SMD:C_1206_3216Metric_Pad1.33x1.80mm_HandSolder, B.Cu at (79.0, 39.0)
- added C12: 100nF, Capacitor_SMD:C_1206_3216Metric_Pad1.33x1.80mm_HandSolder, B.Cu at (88.5, 31.6)
- added C2: 100nF, Capacitor_SMD:C_1206_3216Metric_Pad1.33x1.80mm_HandSolder, B.Cu at (50.0, 39.0)
- added C3: 100u, _MyFootprints:CP_LYING_11x6_2,5mm, F.Cu at (48.8, 38.7)
- added C4: 100nF, Capacitor_SMD:C_1206_3216Metric_Pad1.33x1.80mm_HandSolder, B.Cu at (54.5, 76.0)
- added C5: 100nF, Capacitor_SMD:C_1206_3216Metric_Pad1.33x1.80mm_HandSolder, B.Cu at (47.5, 64.0)
- added C6: 100nF, Capacitor_SMD:C_1206_3216Metric_Pad1.33x1.80mm_HandSolder, B.Cu at (53.0, 64.0)
- added C7: 100nF, Capacitor_SMD:C_1206_3216Metric_Pad1.33x1.80mm_HandSolder, B.Cu at (60.5, 57.1)
- added C8: 100nF, Capacitor_SMD:C_1206_3216Metric_Pad1.33x1.80mm_HandSolder, B.Cu at (60.5, 60.5)
- added C9: 100nF, Capacitor_SMD:C_1206_3216Metric_Pad1.33x1.80mm_HandSolder, B.Cu at (88.0, 73.0)
- added D1: BZT52Bxx, Diode_SMD:D_SOD-123F, B.Cu at (89.0, 60.0)
- added G***: LOGO, _MyFootprints:Logo_GruzaiGarage, F.Cu at (69.0, 20.5)
- added J6: ECU, _MyFootprints:15EDGVC-3.5-05P, B.Cu at (47.0, 42.0)
- added R10: 4k7, Resistor_SMD:R_0805_2012Metric_Pad1.20x1.40mm_HandSolder, B.Cu at (74.0, 52.5)
- added R11: 22R, Resistor_SMD:R_0805_2012Metric_Pad1.20x1.40mm_HandSolder, B.Cu at (88.0, 68.5)
- added R12: 0R, Resistor_SMD:R_0805_2012Metric_Pad1.20x1.40mm_HandSolder, B.Cu at (63.0, 66.0)
- added R13: 0R, Resistor_SMD:R_0805_2012Metric_Pad1.20x1.40mm_HandSolder, B.Cu at (60.5, 66.0)
- added R14: 0R / NC, Resistor_SMD:R_0805_2012Metric_Pad1.20x1.40mm_HandSolder, B.Cu at (57.0, 79.0)
- added R15: 0R / NC, Resistor_SMD:R_0805_2012Metric_Pad1.20x1.40mm_HandSolder, B.Cu at (57.0, 81.5)
- added R16: 0R / NC, Resistor_SMD:R_0805_2012Metric_Pad1.20x1.40mm_HandSolder, B.Cu at (84.0, 74.5)
- added R17: 0R / NC, Resistor_SMD:R_0805_2012Metric_Pad1.20x1.40mm_HandSolder, B.Cu at (84.0, 71.5)
- added R3: 22R, Resistor_SMD:R_0805_2012Metric_Pad1.20x1.40mm_HandSolder, B.Cu at (86.0, 50.5)
- added R4: 22R, Resistor_SMD:R_0805_2012Metric_Pad1.20x1.40mm_HandSolder, B.Cu at (72.0, 46.5)
- added R5: 22R, Resistor_SMD:R_0805_2012Metric_Pad1.20x1.40mm_HandSolder, B.Cu at (72.0, 41.5)
- added R6: 22R, Resistor_SMD:R_0805_2012Metric_Pad1.20x1.40mm_HandSolder, B.Cu at (72.0, 44.0)
- added R7: 0R / NC, Resistor_SMD:R_0805_2012Metric_Pad1.20x1.40mm_HandSolder, B.Cu at (87.5, 38.5)
- added R8: 0R / NC, Resistor_SMD:R_0805_2012Metric_Pad1.20x1.40mm_HandSolder, B.Cu at (87.5, 41.0)
- added R9: 4k7, Resistor_SMD:R_0805_2012Metric_Pad1.20x1.40mm_HandSolder, B.Cu at (71.0, 52.5)
- moved U1 8.54 mm to (53.0, 70.0)
- moved R2 6.26 mm to (86.5, 64.5), turned to 90 degrees
- moved R1 2.55 mm to (71.0, 64.0)
- moved XA1 2.06 mm to (75.5, 70.6)
Connections:
- J1 pad 1: unconnected-(J1-Pin_1-Pad1) -> Net-(D1-K)
- J1 pad 2: unconnected-(J1-Pin_2-Pad2) -> GND
- J2 pad 1: unconnected-(J2-Pin_1-Pad1) -> DISP_CLK
- J2 pad 2: unconnected-(J2-Pin_2-Pad2) -> DISP_DIN
- J2 pad 3: unconnected-(J2-Pin_3-Pad3) -> DISP_CS
- J3 pad 1: unconnected-(J3-Pin_1-Pad1) -> DISP_RST
- J3 pad 2: unconnected-(J3-Pin_2-Pad2) -> DISP_DC
- J3 pad 3: unconnected-(J3-Pin_3-Pad3) -> Net-(J3-Pin_3)
- J3 pad 4: unconnected-(J3-Pin_4-Pad4) -> GND
- J3 pad 5: unconnected-(J3-Pin_5-Pad5) -> DISP_BL
- J5 pad 1: unconnected-(J5-Pin_1-Pad1) -> Net-(J5-Pin_1)
- J5 pad 2: unconnected-(J5-Pin_2-Pad2) -> GND
- J5 pad 3: unconnected-(J5-Pin_3-Pad3) -> Net-(J5-Pin_3)
- R1 pad 2: unconnected-(R1-Pad2) -> DISP_DIN
- R2 pad 2: unconnected-(R2-Pad2) -> DISP_CLK
- U1 pad 1: unconnected-(U1-C1+-Pad1) -> Net-(U1-C1+)
- U1 pad 10: unconnected-(U1-T2IN-Pad10) -> GND
- U1 pad 11: unconnected-(U1-T1IN-Pad11) -> Net-(U1-T1IN)
- U1 pad 12: unconnected-(U1-R1OUT-Pad12) -> Net-(U1-R1OUT)
- U1 pad 13: unconnected-(U1-R1IN-Pad13) -> ECU_TX
- U1 pad 14: unconnected-(U1-T1OUT-Pad14) -> ECU_RX
- U1 pad 15: unconnected-(U1-GND-Pad15) -> GND
- U1 pad 16: unconnected-(U1-VCC-Pad16) -> Net-(U1-VCC)
- U1 pad 2: unconnected-(U1-VS+-Pad2) -> Net-(U1-VS+)
- U1 pad 3: unconnected-(U1-C1--Pad3) -> Net-(U1-C1-)
- U1 pad 4: unconnected-(U1-C2+-Pad4) -> Net-(U1-C2+)
- U1 pad 5: unconnected-(U1-C2--Pad5) -> Net-(U1-C2-)
- U1 pad 6: unconnected-(U1-VS--Pad6) -> Net-(U1-VS-)
- U1 pad 8: unconnected-(U1-R2IN-Pad8) -> GND
- XA1 pad 3V3: unconnected-(XA1-3.3V-Pad3V3) -> +3.3V
- XA1 pad 5V: unconnected-(XA1-Pad5V) -> +5V
- XA1 pad A2: unconnected-(XA1-PadA2) -> UART_PC_RX
- XA1 pad A3: unconnected-(XA1-PadA3) -> Net-(R3-Pad2)
- XA1 pad A7: unconnected-(XA1-PadA7) -> UART_PC_TX
- XA1 pad D0: unconnected-(XA1-D0_RX0-PadD0) -> UART_ECU_RX
- XA1 pad D1: unconnected-(XA1-D1_TX0-PadD1) -> UART_ECU_TX
- XA1 pad D2: unconnected-(XA1-PadD2) -> Net-(R5-Pad1)
- XA1 pad D3: unconnected-(XA1-PadD3) -> Net-(R6-Pad1)
- XA1 pad D4: unconnected-(XA1-PadD4) -> Net-(R4-Pad1)
- XA1 pad D6: unconnected-(XA1-PadD6) -> SWITCH
- XA1 pad D9: unconnected-(XA1-PadD9) -> SPEED_SENS
- XA1 pad GND1: unconnected-(XA1-GND-PadGND1) -> GND
- XA1 pad GND2: unconnected-(XA1-GND-PadGND2) -> GND

Commit message: pcb dev, looking for better connectors
Parts:
- removed J6: ECU, _MyFootprints:15EDGVC-3.5-05P
- added J4: ECU, Connector_Dsub:DSUB-9_Female_Horizontal_P2.77x2.84mm_EdgePinOffset4.94mm_Housed_MountingHolesOffset7.48mm, F.Cu at (51.8, 49.2)
- added R18: 22R, Resistor_SMD:R_0805_2012Metric_Pad1.20x1.40mm_HandSolder, B.Cu at (69.5, 76.4)
- added R19: 22R, Resistor_SMD:R_0805_2012Metric_Pad1.20x1.40mm_HandSolder, B.Cu at (68.0, 74.4)
- moved G*** 60.0 mm to (69.5, 80.5)
- moved R13 46.8 mm to (74.4, 21.3)
- moved R12 45.6 mm to (71.9, 21.3)
- moved R15 26.7 mm to (79.0, 66.3), turned to -90 degrees
- moved R14 23.3 mm to (76.5, 66.3), turned to -90 degrees
- moved C4 21.5 mm to (75.5, 71.3), turned to 90 degrees
- moved U1 17.3 mm to (70.0, 66.8), turned to 0 degrees
- moved C5 15.6 mm to (61.5, 70.8), turned to 90 degrees
- moved C7 15.0 mm to (64.5, 71.6), turned to -90 degrees
- moved C3 11.7 mm to (57.8, 31.2)
- moved C2 11.4 mm to (59.0, 32.0)
- moved C1 10.5 mm to (72.0, 38.5)
- moved C10 10.5 mm to (78.5, 53.5)
- moved C11 10.5 mm to (78.5, 28.5)
- moved R1 10.5 mm to (70.5, 53.5)
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Routing:
- net GND: track 0.00 -> 17.6 mm
- net Net-(U1-VCC): track 0.00 -> 12.6 mm
- net ECU_TX: track 0.00 -> 9.29 mm
- net ECU_RX: track 0.00 -> 9.26 mm
- net Net-(J3-Pin_3): track 0.00 -> 7.88 mm
- net Net-(U1-T1IN): track 0.00 -> 7.78 mm
- net Net-(U1-R1OUT): track 0.00 -> 7.46 mm
- net Net-(U1-C2-): track 0.00 -> 7.32 mm
- net Net-(U1-C1+): track 0.00 -> 6.49 mm
- net Net-(U1-C1-): track 0.00 -> 6.25 mm
- net Net-(J5-Pin_1): track 0.00 -> 5.98 mm
- net SWITCH: track 0.00 -> 5.68 mm
- net Net-(D1-K): track 0.00 -> 3.83 mm
- net Net-(U1-VS-): track 0.00 -> 3.42 mm
- net Net-(U1-C2+): track 0.00 -> 3.23 mm
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