File: pcb/CarDisplay/CarDisplay.kicad_pcb (KiCad board)
At the start: 2 copper layers, 52.5 x 70 mm, 44 parts, among them J1 Switch, J2 Display1, J3 Display2, J4 ECU, J5 SpeedSensor, U1 MAX3232

Commit message: readme
Parts:
- removed J4: ECU, Connector_Dsub:DSUB-9_Female_Horizontal_P2.77x2.84mm_EdgePinOffset4.94mm_Housed_MountingHolesOffset7.48mm
- removed J5: SpeedSensor, _MyFootprints:15EDGVC-3.5-03P
- C3: footprint _MyFootprints:CP_LYING_11x6_2,5mm -> _MyFootprints:CP_LYING_16x10_5,0mm
- J1: value Switch -> ECU; footprint _MyFootprints:15EDGVC-3.5-02P -> Connector_Dsub:DSUB-9_Female_Horizontal_P2.77x2.84mm_EdgePinOffset4.94mm_Housed_MountingHolesOffset7.48mm; moved to F.Cu
- J2: value Display1 -> DISPLAY; footprint _MyFootprints:15EDGVC-3.5-03P -> Connector_Molex:Molex_Mini-Fit_Jr_5569-08A2_2x04_P4.20mm_Horizontal
- J3: value Display2 -> SWITCH&SPEEDSENS; footprint _MyFootprints:15EDGVC-3.5-05P -> Connector_Molex:Molex_Mini-Fit_Jr_5569-06A2_2x03_P4.20mm_Horizontal
- moved J1 42.2 mm to (51.8, 55.4), turned to -90 degrees
- moved J3 19.0 mm to (93.2, 59.0), turned to 90 degrees
- moved R7 11.1 mm to (82.5, 28.5)
- moved C12 11.1 mm to (83.5, 21.6)
- moved R8 11.1 mm to (82.5, 31.1)
- moved J2 10.4 mm to (93.2, 42.1), turned to 90 degrees
- moved D1 7.76 mm to (83.4, 65.4)
- moved C9 5.44 mm to (86.0, 78.1)
- moved R11 5.44 mm to (86.0, 73.6)
- moved R16 5.44 mm to (82.0, 79.6)
- moved R17 5.44 mm to (82.0, 76.6)
- moved R2 5.44 mm to (84.5, 69.6)
- moved C1 3.63 mm to (68.4, 38.8)
- moved C10 3.63 mm to (74.9, 53.8)
- moved C11 3.63 mm to (74.9, 28.8)
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Connections:
- C12 pad 1: Net-(J3-Pin_3) -> Net-(J2-Pin_6)
- C9 pad 1: Net-(J5-Pin_1) -> Net-(J3-Pin_1)
- J1 pad 1: Net-(D1-K) -> +5V
- J1 pad 2: GND -> Net-(J1-Pad2)
- J3 pad 1: DISP_RST -> Net-(J3-Pin_1)
- J3 pad 2: DISP_DC -> GND
- J3 pad 4: GND -> unconnected-(J3-Pin_4-Pad4)
- J3 pad 5: DISP_BL -> Net-(D1-K)
- R11 pad 1: Net-(J5-Pin_3) -> Net-(J3-Pin_3)
- R16 pad 2: Net-(J5-Pin_1) -> Net-(J3-Pin_1)
- R17 pad 2: Net-(J5-Pin_1) -> Net-(J3-Pin_1)
- R18 pad 2: Net-(J4-Pad2) -> Net-(J1-Pad2)
- R19 pad 2: Net-(J4-Pad3) -> Net-(J1-Pad3)
- R7 pad 2: Net-(J3-Pin_3) -> Net-(J2-Pin_6)
- R8 pad 2: Net-(J3-Pin_3) -> Net-(J2-Pin_6)
Routing:
- net Net-(J3-Pin_3): track 7.88 -> 0.00 mm
- net Net-(J2-Pin_6): track 0.00 -> 7.88 mm
- net Net-(J5-Pin_1): track 5.98 -> 0.00 mm
- net Net-(J3-Pin_1): track 0.00 -> 5.98 mm

Commit message: pcb finished
Parts:
- added J4: RX, _MyFootprints:MeasuringPin, F.Cu at (58.6, 31.1)
- added J5: TX, _MyFootprints:MeasuringPin, F.Cu at (55.1, 31.0)
- added J6: RX, _MyFootprints:MeasuringPin, F.Cu at (60.2, 23.6)
- added J7: TX, _MyFootprints:MeasuringPin, F.Cu at (60.2, 20.5)
- added J8: GND, _MyFootprints:MeasuringPin, F.Cu at (57.4, 21.9)
- R14, R15: moved to F.Cu
- moved C12 63.9 mm to (49.1, 75.5), turned to 180 degrees
- moved R7 53.7 mm to (49.7, 71.0)
- moved J2 53.2 mm to (55.5, 79.7), turned to 0 degrees
- moved R8 48.7 mm to (54.3, 70.7), turned to 180 degrees
- moved C5 40.2 mm to (48.6, 32.7)
- moved C6 40.2 mm to (50.1, 28.7)
- moved C7 40.2 mm to (51.6, 33.5)
- moved C8 40.2 mm to (50.1, 25.7)
- moved U1 40.2 mm to (57.1, 28.7)
- moved C4 38.0 mm to (60.1, 36.6), turned to -90 degrees
- moved R19 37.3 mm to (56.4, 39.0), turned to -90 degrees
- moved R18 33.5 mm to (60.3, 44.2), turned to -90 degrees
- moved R14 33.3 mm to (57.5, 39.0), turned to 90 degrees
- moved R15 33.3 mm to (60.0, 39.0), turned to 90 degrees
- moved R9 29.8 mm to (82.9, 67.4), turned to 0 degrees
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Connections:
- C12 pad 1: Net-(J2-Pin_6) -> Net-(J2-Pin_5)
- J2 pad 1: DISP_CLK -> GND
- J2 pad 3: DISP_CS -> DISP_RST
- J2 pad 4: DISP_RST -> DISP_CS
- J2 pad 5: DISP_DC -> Net-(J2-Pin_5)
- J2 pad 6: Net-(J2-Pin_6) -> DISP_DC
- J2 pad 7: GND -> DISP_BL
- J2 pad 8: DISP_BL -> DISP_CLK
- J3 pad 5: Net-(D1-K) -> GND
- J3 pad 6: GND -> Net-(D1-K)
- R7 pad 2: Net-(J2-Pin_6) -> Net-(J2-Pin_5)
- R8 pad 2: Net-(J2-Pin_6) -> Net-(J2-Pin_5)
- XA1 pad GND1: GND -> unconnected-(XA1-GND-PadGND1)
Routing:
- net GND: track 17.6 -> 258.1 mm, vias 0 -> 12
- net +5V: track 0.00 -> 133.7 mm, vias 0 -> 3
- net +3.3V: track 2.68 -> 76.2 mm, vias 0 -> 6
- net DISP_RST: track 0.00 -> 49.9 mm
- net DISP_BL: track 0.00 -> 45.8 mm
- net SPEED_SENS: track 0.00 -> 40.3 mm, vias 0 -> 1
- net DISP_CS: track 0.00 -> 39.8 mm
- net DISP_DC: track 0.00 -> 38.3 mm
- net SWITCH: track 5.68 -> 37.2 mm, vias 0 -> 1
- net DISP_DIN: track 0.00 -> 24.4 mm
- net DISP_CLK: track 0.00 -> 20.3 mm
- net Net-(U1-R1OUT): track 7.46 -> 24.8 mm
- net Net-(J1-Pad3): track 0.00 -> 16.7 mm
- net Net-(J1-Pad2): track 0.00 -> 14.7 mm
- net Net-(J2-Pin_5): track 0.00 -> 12.4 mm
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- added copper zone on B.Cu, net +3.3V
- added copper zone on F.Cu, net +3.3V
- added copper zone on B.Cu, net +5V
- added copper zone on F.Cu, net +5V
- added copper zone on B.Cu, net GND
- added copper zone on F.Cu, net GND
- added copper zone on B.Cu, net Net-(U1-VCC)
- added copper zone on F.Cu, net Net-(U1-VCC)

Commit message: drc passed
Parts:
- moved G*** 1.53 mm to (89.5, 60.2)
Other:
- board text added: "2024 ver. 1.0"
